Commit message: added docker-novnc

File: ros_ws/src/rbcar_model/robots/rbcar2.urdf.xacro (robot description, xacro)
@@ -16,15 +16,16 @@
 	<!-- Global parameters -->
 	<!-- ***************** -->
-	<xacro:property name="PI" value="3.1415926535897931"/>
+	<xacro:property name="PI" value="3.1415926535897931" />
 	<!-- Wheel parameters -->
-	<xacro:property name="wheel_offset_x" value="0.91131" />    <!-- x,y,z in translation from base_link to the center of the wheel -->
+	<xacro:property name="wheel_offset_x" value="0.91131" />    <!-- x,y,z in translation from base_link
+	to the center of the wheel -->
 	<xacro:property name="wheel_offset_y" value="0.62124" />
 	<xacro:property name="wheel_offset_z" value="0.0" />
 	<!-- Flag to select the high or low quality model -->
-	<xacro:property name="hq" value="true" />
-	<xacro:arg name="prefix" default="robot_"/>
-	<xacro:arg name="gps_longitude" default="39.551218"/>
-	<xacro:arg name="gps_latitude" default="-0.467738"/>
-	<xacro:arg name="gpu" default="true"/>
+	<xacro:property name="hq" value="false" />
+	<xacro:arg name="prefix" default="robot_" />
+	<xacro:arg name="gps_longitude" default="39.551218" />
+	<xacro:arg name="gps_latitude" default="-0.467738" />
+	<xacro:arg name="gpu" default="true" />
 	<!-- *************** -->
 	<!-- Robot Elements -->
@@ -34,14 +35,15 @@
 	<!-- Wheels -->
 	<xacro:front_wheel prefix="$(arg prefix)" lr_prefix="left" fr_prefix="front"
-					lr_reflect="1" fr_reflect="1" parent="$(arg prefix)base_link" />
+		lr_reflect="1" fr_reflect="1" parent="$(arg prefix)base_link" />
 	<xacro:front_wheel prefix="$(arg prefix)" lr_prefix="right" fr_prefix="front"
-					lr_reflect="-1" fr_reflect="1" parent="$(arg prefix)base_link" />
+		lr_reflect="-1" fr_reflect="1" parent="$(arg prefix)base_link" />
 	<xacro:rear_wheel prefix="$(arg prefix)" lr_prefix="left" fr_prefix="rear"
-					lr_reflect="1" fr_reflect="-1" parent="$(arg prefix)base_link" />
+		lr_reflect="1" fr_reflect="-1" parent="$(arg prefix)base_link" />
 	<xacro:rear_wheel prefix="$(arg prefix)" lr_prefix="right" fr_prefix="rear"
-					lr_reflect="-1" fr_reflect="-1" parent="$(arg prefix)base_link" />
+		lr_reflect="-1" fr_reflect="-1" parent="$(arg prefix)base_link" />
 	<!-- Sensors -->
 	<!--
-	<xacro:sensor_rslidar_16 prefix="$(arg prefix)top_3d_laser" parent="$(arg prefix)base_link"  gpu="$(arg gpu)">
+	<xacro:sensor_rslidar_16 prefix="$(arg prefix)top_3d_laser" parent="$(arg prefix)base_link"
+	gpu="$(arg gpu)">
 	  <origin xyz="1.163 0.0 1.602" rpy="0 0.2637 0"/>
 	</xacro:sensor_rslidar_16>
@@ -49,11 +51,14 @@
 		<origin xyz="0.319 0.018 0.676" rpy="0 0 0"/>
 	</xacro:sensor_imu_hector>
-	<xacro:sensor_sick_outdoorscan3 prefix="$(arg prefix)front_laser" parent="$(arg prefix)base_link" prefix_topic="front_laser" min_angle="-1.5" max_angle="1.5" gpu="$(arg gpu)">
+	<xacro:sensor_sick_outdoorscan3 prefix="$(arg prefix)front_laser" parent="$(arg prefix)base_link"
+	prefix_topic="front_laser" min_angle="-1.5" max_angle="1.5" gpu="$(arg gpu)">
 		<origin xyz="2.101 0 0.206" rpy="0 0 0"/>
 	</xacro:sensor_sick_outdoorscan3>
-	<xacro:sensor_hokuyo_utm30lx prefix="$(arg prefix)rear_laser" parent="$(arg prefix)base_link" gpu="$(arg gpu)" prefix_topic="rear_laser">
+	<xacro:sensor_hokuyo_utm30lx prefix="$(arg prefix)rear_laser" parent="$(arg prefix)base_link"
+	gpu="$(arg gpu)" prefix_topic="rear_laser">
       		<origin xyz="-0.42925 0.0 0.24674" rpy="0 0 ${PI}"/>
   	</xacro:sensor_hokuyo_utm30lx>
-	<xacro:sensor_gps prefix="$(arg prefix)gps" parent="$(arg prefix)base_link" gps_latitude="$(arg gps_latitude)" gps_longitude="$(arg gps_longitude)">
+	<xacro:sensor_gps prefix="$(arg prefix)gps" parent="$(arg prefix)base_link" gps_latitude="$(arg
+	gps_latitude)" gps_longitude="$(arg gps_longitude)">
 		<origin xyz="0.491 0 1.503" rpy="0 0 0"/>
 	</xacro:sensor_gps>

File: ros_ws/src/rbcar_model/urdf/wheels/suspension_wheel_v3.urdf.xacro (robot description, xacro)
@@ -132,5 +132,6 @@
         <geometry>
           <!--cylinder radius="${tire_dia / 2}" length="${tire_width}"/-->
-          <mesh filename="package://rbcar_model/meshes/wheels/polaris/right_front_wheel.STL"/>
+          <!-- <mesh filename="package://rbcar_model/meshes/wheels/polaris/right_front_wheel.STL"/> -->
+          <mesh filename="package://rbcar_model/meshes/wheels/rbcar_wheel.stl"/>
         </geometry>
         <material name="tire_mat"/>
